Commit message: Changed 2 urdf files to ensure table appears straight

File: jaco_arm/jaco_description/urdf/jaco_robot.urdf (robot description, URDF)
Before this commit: robot JacoOnTable, 31 links, 30 joints
Links:
- removed link arm_stand
- removed link robot_base
- removed link table_base
- removed link table_top
- removed link tabletop_corner
- removed link tabletop_ontop
- removed link world
- added link robot_root
- link jaco_0_baseA: mass 0.2844 -> 0.5688
- link jaco_0_baseB_limb: mass 0.2576 -> 0.5152
- link jaco_1_shoulder_limb: mass 0.2391 -> 0.4782
- link jaco_2_upperarm_limb: mass 0.685815 -> 1.37163
- link jaco_3_forearm_limb: mass 0.337964595 -> 0.67592919
- link jaco_4_upperwrist_limb: mass 0.12275168143 -> 0.24550336286
- link jaco_5_lowerwrist_limb: mass 0.12275 -> 0.2455
- link jaco_6_hand_limb: mass 0.1 -> 0.2
- link jaco_fingers_base_link: mass 0.0005 -> 0.001
- link jaco_ring_1: mass 0.00436 -> 0.00872
- link jaco_ring_2: mass 0.00436 -> 0.00872
- link jaco_ring_3: mass 0.00436 -> 0.00872
- link jaco_ring_4: mass 0.00338267061984 -> 0.00676534123969
- link jaco_ring_5: mass 0.00338267061984 -> 0.00676534123969
- link jaco_ring_6: mass 0.00338 -> 0.00676
Joints:
- removed joint base_to_jaco_on_table
- removed joint j1
- removed joint j2b
- removed joint set_tabletop_relto_corner
- removed joint table_tabletop_totop
- removed joint table_to_arm
- joint jaco_arm_joint: origin xyz=-0.000482247085224208 0.08 -0.000503436190578577 rpy=1.57079632679 0 3.14159265359 -> xyz=0 0 0 rpy=0 0 0; parent arm_stand -> robot_root

File: jaco_tutorial/jaco_on_table/urdf/jaco_on_table_centered.urdf.xacro (robot description, xacro)
@@ -24,6 +24,7 @@
   <xacro:include filename="$(find jaco_on_table)/urdf/objects/table.xacro" />
   <joint name="table_to_arm" type="fixed">
-    <origin xyz="0.40488474042 0.27988474042 0.3" rpy="0 0 -0.785398163397458" />
-    <origin xyz="0.40488474042 0.27988474042 0.3" rpy="0 0 0"/>
+    <!--origin xyz="0.40488474042 0.27988474042 0.3" rpy="0 0 -0.785398163397458" /-->
+    <!--removed rotation from table and centered table-->
+    <origin xyz="0 0 0.3" rpy="0 0 0"/>
     <parent link="robot_base"/>
     <child link="table_base"/>
@@ -39,4 +40,5 @@
   <xacro:jaco_arm parent="arm_stand" mass_divider="2" finger_mass_divider="1">
     <origin xyz="-0.000482247085224208 0.08 -0.000503436190578577" rpy="1.57079632679 0 3.14159265359" />
+    <!--origin xyz="-0 0 0.1" rpy="0 0 0" /-->
     <xacro:arg name="add_transmission_pos" default="$(arg add_transmission_pos)"/>
     <xacro:arg name="add_transmission_vel" default="$(arg add_transmission_vel)"/>

File: jaco_tutorial/jaco_on_table/urdf/jaco_on_table_robot_gazebo_ctrl.urdf.xacro (robot description, xacro)
@@ -16,5 +16,5 @@
     </link>
 -->
-    <xacro:include filename="$(find jaco_on_table)/urdf/jaco_on_table.urdf.xacro">
+    <xacro:include filename="$(find jaco_on_table)/urdf/jaco_on_table_centered.urdf.xacro">
         <xacro:arg name="add_transmission_pos" default="$(arg add_transmission_pos)"/>
         <xacro:arg name="add_transmission_vel" default="$(arg add_transmission_vel)"/>
